File: kicad/MHI-AC-CTRL/MHI-AC-CTRL.kicad_pcb (KiCad board)
At the start: 2 copper layers, 41.9 x 27.2 mm, 9 parts, among them J1 Conn_01x05, J3 Conn_01x03, U1 TSR_1-2450, U2 WeMos_D1_mini, U3 LEVEL-SHIFTER-4CH

Commit message: Resizing the board to fit for model SKR ZSX model where we have capacitor top right Following suggestion under https://github.com/absalom-muc/MHI-AC-Ctrl/issues/56
Parts:
- moved J3 1.58 mm to (85.8, 44.9)
Routing:
- net GND: track 84.7 -> 86.5 mm
- net DS18x20: track 25.5 -> 24.2 mm
- net +3V3: track 67.0 -> 65.7 mm
- added copper zone on B.Cu, net GND
- added copper zone on F.Cu, net GND
Other:
- outline, holes or cut-outs redrawn
- board text added: "Feb'23"
- board text added: "MHI-AC-Ctrl m.ZSX"
- board text removed: "MHI-AC-Ctrl v2.3"
- board text removed: "Oktober 2022"
Changed lines of the file:
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@@
       (disableapertmacros false)
       (usegerberextensions true)
-      (usegerberattributes true)
-      (usegerberadvancedattributes true)
+      (usegerberattributes false)
+      (usegerberadvancedattributes false)
       (creategerberjobfile false)
       (svguseinch false)
@@
       (psa4output false)
       (plotreference true)
-      (plotvalue false)
+      (plotvalue true)
       (plotinvisibletext false)
       (sketchpadsonfab false)
-      (subtractmaskfromsilk true)
+      (subtractmaskfromsilk false)
       (outputformat 1)
       (mirror false)
@@
   )
   (footprint "Connector_JST:JST_XH_B3B-XH-A_1x03_P2.50mm_Vertical" (layer "F.Cu")
-    (at 84.3236 44.45 90)
+    (at 85.835 44.918 90)
     (descr "JST XH series connector, B3B-XH-A (http://www.jst-mfg.com/product/pdf/eng/eXH.pdf), generated with kicad-footprint-generator")
     (tags "connector JST XH vertical")
@@
   (gr_line (start 85.49 49.51) (end 86.24 49.51) (layer "B.SilkS") (width 0.15))
   (gr_line (start 85.49 49.51) (end 85.5 47.71) (layer "B.SilkS") (width 0.15))
+  (gr_line (start 83.058 46.228) (end 83.058 37.084) (layer "Edge.Cuts") (width 0.1))
+  (gr_line (start 79.248 46.228) (end 83.058 46.228) (layer "Edge.Cuts") (width 0.1))
   (gr_line (start 121.158 64.262) (end 79.248 64.262) (layer "Edge.Cuts") (width 0.1))
-  (gr_line (start 79.248 37.084) (end 121.158 37.084) (layer "Edge.Cuts") (width 0.1))
-  (gr_line (start 79.248 64.262) (end 79.248 37.084) (layer "Edge.Cuts") (width 0.1))
+  (gr_line (start 79.248 46.228) (end 79.248 64.262) (layer "Edge.Cuts") (width 0.1))
+  (gr_line (start 83.058 37.084) (end 121.158 37.084) (layer "Edge.Cuts") (width 0.1))
   (gr_line (start 121.158 37.084) (end 121.158 64.262) (layer "Edge.Cuts") (width 0.1))
-  (gr_text "MHI-AC-Ctrl v2.3" (at 111.76 50.8) (layer "B.SilkS")
+  (gr_text "MHI-AC-Ctrl m.ZSX" (at 111.76 50.8) (layer "B.SilkS")
     (effects (font (size 1 1) (thickness 0.15)) (justify mirror))
   )
-  (gr_text "Oktober 2022" (at 110.49 53.34) (layer "B.SilkS")
+  (gr_text "Feb'23" (at 110.49 53.34) (layer "B.SilkS")
     (effects (font (size 1 1) (thickness 0.15)) (justify mirror))
   )
-  (gr_text "MHI-AC-Ctrl v2.3" (at 80.772 55.5244 90) (layer "F.SilkS")
+  (gr_text "MHI-AC-Ctrl m.ZSX" (at 80.772 55.5244 90) (layer "F.SilkS")
     (effects (font (size 1 1) (thickness 0.15)))
+  )
+  (dimension (type aligned) (layer "F.Cu")
+    (pts (xy 79.248 64.262) (xy 121.412 64.262))
+    (height 9.144)
+    (gr_text "42,1640 mm" (at 100.33 71.606) (layer "F.Cu")
+      (effects (font (size 1.5 1.5) (thickness 0.3)))
+    )
+    (format (units 3) (units_format 1) (precision 4))
+    (style (thickness 0.2) (arrow_length 1.27) (text_position_mode 0) (extension_height 0.58642) (extension_offset 0.5) keep_text_aligned)
+  )
+  (dimension (type aligned) (layer "F.Cu")
+    (pts (xy 121.158 37.084) (xy 121.158 64.516))
+    (height -12.446)
+    (gr_text "27,4320 mm" (at 131.804 50.8 90) (layer "F.Cu")
+      (effects (font (size 1.5 1.5) (thickness 0.3)))
+    )
+    (format (units 3) (units_format 1) (precision 4))
+    (style (thickness 0.2) (arrow_length 1.27) (text_position_mode 0) (extension_height 0.58642) (extension_offset 0.5) keep_text_aligned)
   )
   (segment (start 87.63 60.4012) (end 83.917 60.4012) (width 0.5) (layer "B.Cu") (net 1))
@@
   (segment (start 109.22 43.14) (end 109.26 43.18) (width 0.5) (layer "F.Cu") (net 2))
   (segment (start 97.1296 52.7304) (end 99.6696 52.7304) (width 0.5) (layer "F.Cu") (net 2))
+  (segment (start 83.7862 50.2704) (end 87.6516 50.2704) (width 0.5) (layer "B.Cu") (net 2))
   (segment (start 111.76 46.99) (end 111.76 46.228) (width 0.5) (layer "B.Cu") (net 2))
+  (segment (start 87.6516 50.2704) (end 87.884 50.038) (width 0.5) (layer "B.Cu") (net 2))
+  (segment (start 86.4 39.918) (end 85.835 39.918) (width 0.5) (layer "B.Cu") (net 2))
   (segment (start 99.6696 52.7304) (end 111.6076 52.7304) (width 0.5) (layer "B.Cu") (net 2))
   (segment (start 111.6076 52.7304) (end 111.76 52.578) (width 0.5) (layer "B.Cu") (net 2))
@@
   (segment (start 111.76 46.228) (end 109.26 43.728) (width 0.5) (layer "B.Cu") (net 2))
   (segment (start 109.26 43.728) (end 109.26 43.18) (width 0.5) (layer "B.Cu") (net 2))
-  (segment (start 81.026 40.132) (end 81.026 50.292) (width 0.5) (layer "B.Cu") (net 2))
   (segment (start 90.13 61.762) (end 90.13 60.4012) (width 0.5) (layer "B.Cu") (net 2))
-  (segment (start 81.708 39.45) (end 81.026 40.132) (width 0.5) (layer "B.Cu") (net 2))
   (segment (start 81.788 62.484) (end 89.408 62.484) (width 0.5) (layer "B.Cu") (net 2))
   (segment (start 81.026 50.292) (end 81.026 61.722) (width 0.5) (layer "B.Cu") (net 2))
@@
   (segment (start 111.76 46.99) (end 111.76 52.578) (width 0.5) (layer "B.Cu") (net 2))
   (segment (start 89.408 62.484) (end 90.13 61.762) (width 0.5) (layer "B.Cu") (net 2))
+  (segment (start 87.884 50.038) (end 87.884 41.402) (width 0.5) (layer "B.Cu") (net 2))
   (segment (start 90.1192 56.9792) (end 90.1192 60.3904) (width 0.5) (layer "B.Cu") (net 2))
   (segment (start 111.76 52.578) (end 111.76 57.15) (width 0.5) (layer "B.Cu") (net 2))
   (segment (start 90.1192 60.3904) (end 90.13 60.4012) (width 0.5) (layer "B.Cu") (net 2))
-  (segment (start 84.3236 39.45) (end 81.708 39.45) (width 0.5) (layer "B.Cu") (net 2))
   (segment (start 81.026 61.722) (end 81.788 62.484) (width 0.5) (layer "B.Cu") (net 2))
+  (segment (start 87.884 41.402) (end 86.4 39.918) (width 0.5) (layer "B.Cu") (net 2))
   (segment (start 109.22 46.482) (end 109.22 46.99) (width 0.5) (layer "F.Cu") (net 3))
   (segment (start 111.76 43.942) (end 109.22 46.482) (width 0.5) (layer "F.Cu") (net 3))
@@
   (segment (start 83.7862 57.7704) (end 86.5016 57.7704) (width 0.25) (layer "F.Cu") (net 6))
   (segment (start 96.012 48.26) (end 101.6 48.26) (width 0.25) (layer "F.Cu") (net 6))
+  (segment (start 91.44 44.958) (end 85.875 44.958) (width 0.5) (layer "F.Cu") (net 7))
+  (segment (start 85.875 44.958) (end 85.835 44.918) (width 0.5) (layer "F.Cu") (net 7))
+  (segment (start 93.98 43.815) (end 92.583 43.815) (width 0.5) (layer "F.Cu") (net 7))
   (segment (start 109.22 58.42) (end 111.76 60.96) (width 0.5) (layer "F.Cu") (net 7))
-  (segment (start 92.583 43.815) (end 93.98 43.815) (width 0.5) (layer "F.Cu") (net 7))
+  (segment (start 92.583 43.815) (end 91.44 44.958) (width 0.5) (layer "F.Cu") (net 7))
   (segment (start 109.22 57.15) (end 109.22 58.42) (width 0.5) (layer "F.Cu") (net 7))
-  (segment (start 84.3236 44.45) (end 91.948 44.45) (width 0.5) (layer "F.Cu") (net 7))
-  (segment (start 91.948 44.45) (end 92.583 43.815) (width 0.5) (layer "F.Cu") (net 7))
   (segment (start 111.76 60.96) (end 111.76 62.23) (width 0.5) (layer "F.Cu") (net 7))
   (segment (start 93.98 43.815) (end 93.98 42.672) (width 0.5) (layer "B.Cu") (net 7))
@@
   (segment (start 115.824 62.23) (end 111.76 62.23) (width 0.5) (layer "B.Cu") (net 7))
   (segment (start 119.38 45.72) (end 119.38 58.674) (width 0.5) (layer "B.Cu") (net 7))
+  (segment (start 85.852 42.418) (end 85.835 42.418) (width 0.25) (layer "F.Cu") (net 8))
   (segment (start 101.6 41.91) (end 101.6 39.37) (width 0.25) (layer "F.Cu") (net 8))
   (segment (start 91.44 40.005) (end 93.345 41.91) (width 0.25) (layer "F.Cu") (net 8))
-  (segment (start 84.3236 41.95) (end 86.32 41.95) (width 0.25) (layer "F.Cu") (net 8))
+  (segment (start 88.265 40.005) (end 85.852 42.418) (width 0.25) (layer "F.Cu") (net 8))
   (segment (start 93.345 41.91) (end 101.6 41.91) (width 0.25) (layer "F.Cu") (net 8))
   (segment (start 104.14 42.545) (end 103.505 41.91) (width 0.25) (layer "F.Cu") (net 8))
   (segment (start 88.265 40.005) (end 91.44 40.005) (width 0.25) (layer "F.Cu") (net 8))
-  (segment (start 86.32 41.95) (end 88.265 40.005) (width 0.25) (layer "F.Cu") (net 8))
   (segment (start 103.505 41.91) (end 101.6 41.91) (width 0.25) (layer "F.Cu") (net 8))
   (segment (start 104.14 43.815) (end 104.14 42.545) (width 0.25) (layer "F.Cu") (net 8))
@@
   (segment (start 101.6 56.642) (end 102.87 55.372) (width 0.25) (layer "F.Cu") (net 14))
   (segment (start 101.6 62.23) (end 101.6 56.642) (width 0.25) (layer "F.Cu") (net 14))
+  (zone (net 2) (net_name "GND") (layer "F.Cu") (hatch edge 0.508)
+    (connect_pads (clearance 0.508))
+    (min_thickness 0.254) (filled_areas_thickness no)
+    (fill yes (mode hatch) (thermal_gap 0.508) (thermal_bridge_width 0.508)
+      (hatch_thickness 0.254) (hatch_gap 0.254) (hatch_orientation 0)
+      (hatch_border_algorithm hatch_thickness) (hatch_min_hole_area 0.3))
+    (polygon
+      (pts
+        (xy 121.158 64.516)
+        (xy 79.248 64.262)
+        (xy 79.248 46.228)
+        (xy 83.058 46.228)
+        (xy 83.058 37.084)
+        (xy 121.158 37.084)
+      )
+    )
+  )
+  (zone (net 2) (net_name "GND") (layer "B.Cu") (hatch edge 0.508)
+    (connect_pads (clearance 0.508))
+    (min_thickness 0.254) (filled_areas_thickness no)
+    (fill yes (mode hatch) (thermal_gap 0.508) (thermal_bridge_width 0.508)
+      (hatch_thickness 0.254) (hatch_gap 0.254) (hatch_orientation 0)
+      (hatch_border_algorithm hatch_thickness) (hatch_min_hole_area 0.3))
+    (polygon
+      (pts
+        (xy 121.158 64.262)
+        (xy 79.248 64.262)
+        (xy 79.248 46.228)
+        (xy 83.058 46.228)
+        (xy 83.058 37.084)
+        (xy 121.158 37.084)
+      )
+    )
+  )
 )
